File: 648-Artur(projetos eletronicos)/AudioAmp60W/AudioAmp60W/AudioAmp60W/AudioAmp60W.kicad_sch (KiCad schematic)
At the start: 66 parts, among them J1 in, J2 Screw_Terminal_01x03, Q10 BC550, Q11 BC560, Q12 BC550, Q13 BC560, Q14 BDW93, Q2 BC550, Q3 BC560, Q4 BDW94, Q5 BC550, Q6 BC560, Q7 BC560, Q8 BC550, Q9 BC550

Commit message: Add files via upload
Parts:
- Sound1: value in -> out
Changed lines of the file:
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@@
 		)
 		(property "Value" "BC550"
-			(at 119.634 121.158 0)
+			(at 117.602 121.158 0)
 			(effects
 				(font
@@
 			)
 		)
-		(property "Value" "in"
+		(property "Value" "out"
 			(at 254 101.5999 0)
 			(effects
